Commit message: Added new world and added navigation capatabilities

File: urdf/model.urdf.xacro (robot description, xacro)
@@ -1,4 +1,8 @@
 <?xml version="1.0"?>
-<robot name="field_robot" xmlns:xacro="http://ros.org/wiki/xacro">
+<robot xmlns:sensor="http://playerstage.sourceforge.net/gazebo/xmlschema/#sensor"
+       xmlns:controller="http://playerstage.sourceforge.net/gazebo/xmlschema/#controller"
+       xmlns:interface="http://playerstage.sourceforge.net/gazebo/xmlschema/#interface"
+       xmlns:xacro="http://ros.org/wiki/xacro"
+		name="field_robot_model">
 	<xacro:property name="wheel_diameter" value="0.15"/>
 	<xacro:property name="wheel_depth" value="0.05"/>
@@ -6,6 +10,6 @@
 	<xacro:property name="wheel_x_pos" value="0.175"/>
 	<xacro:property name="box_h" value="0.125"/>
-	<xacro:property name="z_offset" value="${0.5*box_h+0.0275}"/>
-	<xacro:property name="laser_offset" value="0.18"/>
+	<xacro:property name="z_offset_" value="${0.5*box_h+0.055}"/>
+	<xacro:property name="laser_offset" value="0.24"/>
  	<xacro:macro name="default_inertial" params="mass">
     	<inertial>
@@ -42,5 +46,5 @@
 			<child link="${prefix}_wheel"/>
 			<axis xyz="0 0 1"/>
-			<origin rpy="0 1.57 1.57" xyz="${h_refl*wheel_y_pos} ${v_refl*wheel_x_pos} ${z_offset-0.0275}"/>
+			<origin rpy="0 1.57 1.57" xyz="${h_refl*wheel_y_pos} ${v_refl*wheel_x_pos+v_refl*0.01} ${z_offset_-0.0275}"/>
 		</joint>
 		<transmission name="${prefix}_trans">
@@ -67,5 +71,5 @@
 					<cylinder length="0.04" radius="0.02"/>
 				</geometry>
-				<origin rpy="0 0 0" xyz="${h_refl*0.2} ${v_refl*0.1075} ${z_offset+0.0825}"/>
+				<origin rpy="0 0 0" xyz="${h_refl*0.2} ${v_refl*0.1075} ${z_offset_+0.0825}"/>
 			</visual>
 			<collision>
@@ -73,5 +77,5 @@
 					<cylinder length="0.04" radius="0.02"/>
 				</geometry>
-				<origin rpy="0 0 0" xyz="${h_refl*0.2} ${v_refl*0.1075} ${z_offset+0.0825}"/>
+				<origin rpy="0 0 0" xyz="${h_refl*0.2} ${v_refl*0.1075} ${z_offset_+0.0825}"/>
 			</collision>
 			<xacro:default_inertial mass="1"/>
@@ -87,5 +91,5 @@
 				<box size="0.6 .3 .125"/>
 			</geometry>
-			<origin rpy="0 0 0" xyz="0.0 0.0 ${z_offset}"/>
+			<origin rpy="0 0 0" xyz="0.0 0.0 ${z_offset_}"/>
 		</visual>
 		<collision>
@@ -93,6 +97,7 @@
 				<box size="0.6 .3 .125"/>
 			</geometry>
-			<origin rpy="0 0 0" xyz="0.0 0.0 ${z_offset}"/>
+			<origin rpy="0 0 0" xyz="0.0 0.0 ${z_offset_}"/>
 		</collision>
+		<xacro:default_inertial mass="20"/>
 	</link>
 	<xacro:wheel prefix="left_front" h_refl="1" v_refl="1"/>
@@ -109,5 +114,5 @@
 				<box size="0.6 .3 .03"/>
 			</geometry>
-			<origin rpy="0 0 0" xyz="0 0 ${z_offset+0.1175}"/>
+			<origin rpy="0 0 0" xyz="0 0 ${z_offset_+0.1175}"/>
 		</visual>
 		<xacro:default_inertial mass="10"/>
@@ -117,27 +122,15 @@
 		<child link="top_plate"/>
 	</joint>
-    <link name="laser">
-		<visual>
-			<geometry>
-				<mesh filename="package://sick_tim/meshes/sick_tim310.stl"/>
-			</geometry>
-			<material name="black"/>
-		</visual>
-      <inertial>
-        <mass value="0.001" />
-        <origin xyz="0 0 0" />
-        <inertia ixx="0.000001" ixy="0.0" ixz="0.0"
-          iyy="0.000001" iyz="0.0" izz="0.000001" />
-      </inertial>
-    </link>
-    <joint name="laser_mount_joint" type="fixed">
-      <parent link="base_link" />
-      <child link="laser" />
-      <origin rpy="0 3.14 -1.57" xyz="0 0 ${laser_offset}"/>
-    </joint>
-  <gazebo>
+  <xacro:include filename="$(find sick_tim)/urdf/sick_tim.urdf.xacro" />
+  <xacro:sick_tim310 name="laser" ros_topic="gazebo/scan"  />
+<gazebo>
     <plugin name="gazebo_ros_control" filename="libgazebo_ros_control.so">
       <robotNamespace>/</robotNamespace>
     </plugin>
   </gazebo>
+      <joint name="laser_base_joint" type="fixed">
+      <parent link="base_link" />
+      <child link="laser_mount_link" />
+      <origin rpy="0 3.14 3.14" xyz="0 0 ${laser_offset}"/>
+    </joint>
 </robot>

Commit message: Updated version

File: urdf/model.urdf.xacro (robot description, xacro)
@@ -4,5 +4,5 @@
        xmlns:interface="http://playerstage.sourceforge.net/gazebo/xmlschema/#interface"
        xmlns:xacro="http://ros.org/wiki/xacro"
-		name="field_robot_model">
+		name="field_robot">
 	<xacro:property name="wheel_diameter" value="0.15"/>
 	<xacro:property name="wheel_depth" value="0.05"/>
@@ -46,5 +46,5 @@
 			<child link="${prefix}_wheel"/>
 			<axis xyz="0 0 1"/>
-			<origin rpy="0 1.57 1.57" xyz="${h_refl*wheel_y_pos} ${v_refl*wheel_x_pos+v_refl*0.01} ${z_offset_-0.0275}"/>
+			<origin rpy="1.57 0 0" xyz="${h_refl*wheel_y_pos} ${v_refl*wheel_x_pos+v_refl*0.01} ${z_offset_-0.0275}"/>
 		</joint>
 		<transmission name="${prefix}_trans">
@@ -55,4 +55,5 @@
  		 	<actuator name="${prefix}_motor">
    			 	<mechanicalReduction>1</mechanicalReduction>
+				<hardwareInterface>VelocityJointInterface</hardwareInterface>
   			</actuator>
 		</transmission>
@@ -99,5 +100,4 @@
 			<origin rpy="0 0 0" xyz="0.0 0.0 ${z_offset_}"/>
 		</collision>
-		<xacro:default_inertial mass="20"/>
 	</link>
 	<xacro:wheel prefix="left_front" h_refl="1" v_refl="1"/>
@@ -124,9 +124,4 @@
   <xacro:include filename="$(find sick_tim)/urdf/sick_tim.urdf.xacro" />
   <xacro:sick_tim310 name="laser" ros_topic="gazebo/scan"  />
-<gazebo>
-    <plugin name="gazebo_ros_control" filename="libgazebo_ros_control.so">
-      <robotNamespace>/</robotNamespace>
-    </plugin>
-  </gazebo>
       <joint name="laser_base_joint" type="fixed">
       <parent link="base_link" />
@@ -134,3 +129,15 @@
       <origin rpy="0 3.14 3.14" xyz="0 0 ${laser_offset}"/>
     </joint>
+<gazebo>
+    <plugin name="gazebo_ros_control" filename="libgazebo_ros_control.so">
+      <robotNamespace>/field_robot</robotNamespace>
+	  <robotSimType>gazebo_ros_control/DefaultRobotHWSim</robotSimType>
+    </plugin>
+<plugin name="joint_state_publisher" filename="libgazebo_ros_joint_state_publisher.so">
+      <robotNamespace>/field_robot</robotNamespace>
+      <jointName>left_back_wheel_joint, left_front_wheel_joint, right_back_wheel_joint, right_back_wheel_joint</jointName>
+      <updateRate>100.0</updateRate>
+     <alwaysOn>true</alwaysOn>
+      </plugin>
+  </gazebo>
 </robot>

File: urdf/urdfwithwheels.urdf.xacro (robot description, xacro)
@@ -46,5 +46,5 @@
 			<child link="${prefix}_wheel"/>
 			<axis xyz="0 0 1"/>
-			<origin rpy="1.57 0 0" xyz="${h_refl*wheel_y_pos} ${v_refl*wheel_x_pos+v_refl*0.01} ${z_offset_-0.0275}"/>
+			<origin rpy="0 1.57 1.57" xyz="${h_refl*wheel_y_pos} ${v_refl*wheel_x_pos+v_refl*0.01} ${z_offset_-0.0275}"/>
 		</joint>
 		<transmission name="${prefix}_trans">
@@ -134,10 +134,4 @@
 	  <robotSimType>gazebo_ros_control/DefaultRobotHWSim</robotSimType>
     </plugin>
-<plugin name="joint_state_publisher" filename="libgazebo_ros_joint_state_publisher.so">
-      <robotNamespace>/field_robot</robotNamespace>
-      <jointName>chassis_swivel_joint, swivel_wheel_joint, left_hub_joint, right_hub_joint</jointName>
-      <updateRate>100.0</updateRate>
-     <alwaysOn>true</alwaysOn>
-      </plugin>
   </gazebo>
 </robot>

Commit message: Added worlds for simulation causes

File: urdf/model.urdf.xacro (robot description, xacro)
@@ -46,5 +46,5 @@
 			<child link="${prefix}_wheel"/>
 			<axis xyz="0 0 1"/>
-			<origin rpy="1.57 0 0" xyz="${h_refl*wheel_y_pos} ${v_refl*wheel_x_pos+v_refl*0.01} ${z_offset_-0.0275}"/>
+			<origin rpy="0 1.57 1.57" xyz="${h_refl*wheel_y_pos} ${v_refl*wheel_x_pos+v_refl*0.01} ${z_offset_-0.0275}"/>
 		</joint>
 		<transmission name="${prefix}_trans">
@@ -100,4 +100,5 @@
 			<origin rpy="0 0 0" xyz="0.0 0.0 ${z_offset_}"/>
 		</collision>
+		<xacro:default_inertial mass="20"/>
 	</link>
 	<xacro:wheel prefix="left_front" h_refl="1" v_refl="1"/>
@@ -131,13 +132,7 @@
 <gazebo>
     <plugin name="gazebo_ros_control" filename="libgazebo_ros_control.so">
-      <robotNamespace>/field_robot</robotNamespace>
+      <robotNamespace>/</robotNamespace>
 	  <robotSimType>gazebo_ros_control/DefaultRobotHWSim</robotSimType>
     </plugin>
-<plugin name="joint_state_publisher" filename="libgazebo_ros_joint_state_publisher.so">
-      <robotNamespace>/field_robot</robotNamespace>
-      <jointName>left_back_wheel_joint, left_front_wheel_joint, right_back_wheel_joint, right_back_wheel_joint</jointName>
-      <updateRate>100.0</updateRate>
-     <alwaysOn>true</alwaysOn>
-      </plugin>
   </gazebo>
 </robot>
